File: pcb/clockradio/_autosave-clockradio.kicad_sch (KiCad schematic)
At the start: 10 parts, among them J1 CUE_SJ1-352XNG, SW1(Left)1 SW_Push, SW2(Right)1 SW_Push, SW3(Select)1 SW_Push, SW4(Mode)1 SW_Push, U1 RDA5807M_Module, U2 RPi_Pico_TH

Commit message: update
Parts:
- renumbered SW1(Left)1 to SW1(Right)1, SW2(Right)1 to SW2(Left)1
Changed lines of the file:
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@@
   (symbol (lib_id "Switch:SW_Push") (at 73.66 64.77 0) (unit 1)
     (in_bom yes) (on_board yes) (fields_autoplaced)
-    (property "Reference" "SW1(Left)1" (id 0) (at 73.66 57.15 0))
+    (property "Reference" "SW1(Right)1" (id 0) (at 73.66 57.15 0))
     (property "Value" "SW_Push" (id 1) (at 73.66 59.69 0))
     (property "Footprint" "Button_Switch_THT:SW_PUSH_6mm_H8mm" (id 2) (at 73.66 59.69 0)
@@
   (symbol (lib_id "Switch:SW_Push") (at 73.66 73.66 0) (unit 1)
     (in_bom yes) (on_board yes) (fields_autoplaced)
-    (property "Reference" "SW2(Right)1" (id 0) (at 73.66 66.04 0))
+    (property "Reference" "SW2(Left)1" (id 0) (at 73.66 66.04 0))
     (property "Value" "SW_Push" (id 1) (at 73.66 68.58 0))
     (property "Footprint" "Button_Switch_THT:SW_PUSH_6mm_H8mm" (id 2) (at 73.66 68.58 0)
@@
     )
     (path "/89536d73-f188-4720-96c4-ab4ddf531371"
-      (reference "SW1(Left)1") (unit 1) (value "SW_Push") (footprint "Button_Switch_THT:SW_PUSH_6mm_H8mm")
+      (reference "SW1(Right)1") (unit 1) (value "SW_Push") (footprint "Button_Switch_THT:SW_PUSH_6mm_H8mm")
     )
     (path "/92a38e0a-070a-4048-8d27-ea836f157e34"
-      (reference "SW2(Right)1") (unit 1) (value "SW_Push") (footprint "Button_Switch_THT:SW_PUSH_6mm_H8mm")
+      (reference "SW2(Left)1") (unit 1) (value "SW_Push") (footprint "Button_Switch_THT:SW_PUSH_6mm_H8mm")
     )
     (path "/a30be8ea-33ab-475b-b7ab-56547d20c54b"
